File: AltoidsPCB.kicad_pcb (KiCad board)
At the start: 2 copper layers, 91.4 x 50.8 mm, 144 parts, among them J1 Conn_01x05_Male, J2 Conn_01x26_Male, J3 Conn_01x01_Male

Commit message: update to Kicad 6
Other:
- net class Default removed
